File: 411 Final Schematic.sch (EAGLE design)
At the start: 10 parts, among them Q1 16MHz, U1 ATMEGA328P-PU

Commit message: Add files via upload
Other:
- note added: "Generate the Clock for the ATMega328"
- note added: "The ATMega processor will take the inputs (photocell) to control output (Servo Motor)."
- note added: "The photoresistor will detect change in light."
- note added: "The servo motor will receive a signal from the processor."
- note added: "The voltage will apply power to all components."
Changed lines of the file:
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@@
 <sheet>
 <plain>
+<text x="15.24" y="53.34" size="1.778" layer="91">The voltage will apply power to all components.</text>
+<text x="139.7" y="48.26" size="1.778" layer="91" rot="R90">The photoresistor will detect change in light.</text>
+<text x="68.58" y="81.28" size="1.778" layer="91">The servo motor will receive a signal from the processor.</text>
+<text x="53.34" y="17.78" size="1.778" layer="91">The ATMega processor will take the inputs (photocell) to control output (Servo Motor).</text>
+<text x="27.94" y="27.94" size="1.778" layer="91">Generate the Clock for the ATMega328</text>
 </plain>
 <instances>

Commit message: Add files via upload
Other:
- note added: "- Servo Motor"
- note added: "Date: 12/04/2020 7:10 PM"
- note added: "Document Number: Final Schematic"
- note added: "Notes VCC=9V Inputs: - Photoresistor - Voltage Outputs:"
- note added: "Team 14: Mai Her Prachthearat Ngoy Naiqi Yao Uzias Cruz"
- note added: "Title: ECE411 Automatic Bird Feeder"
Changed lines of the file:
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@@
 <text x="53.34" y="17.78" size="1.778" layer="91">The ATMega processor will take the inputs (photocell) to control output (Servo Motor).</text>
 <text x="27.94" y="27.94" size="1.778" layer="91">Generate the Clock for the ATMega328</text>
+<text x="149.86" y="10.16" size="1.778" layer="95">Team 14:
+Mai Her
+Prachthearat Ngoy
+Naiqi Yao
+Uzias Cruz</text>
+<text x="149.86" y="27.94" size="1.778" layer="95">Title: ECE411
+Automatic Bird Feeder</text>
+<text x="149.86" y="5.08" size="1.778" layer="95">Date: 12/04/2020 7:10 PM</text>
+<text x="177.8" y="17.78" size="1.778" layer="95">Document Number:
+Final Schematic</text>
+<text x="149.86" y="58.42" size="1.778" layer="95">Notes
+VCC=9V
+Inputs:
+- Photoresistor
+- Voltage
+Outputs:</text>
+<text x="149.86" y="55.88" size="1.778" layer="95">- Servo Motor</text>
 </plain>
 <instances>
@@
 </drawing>
 <compatibility>
+<note version="6.3" minversion="6.2.2" severity="warning">
+Since Version 6.2.2 text objects can contain more than one line,
+which will not be processed correctly with this version.
+</note>
 <note version="8.2" severity="warning">
 Since Version 8.2, EAGLE supports online libraries. The ids
